File: Hardware/Kicad/PAL-sign.kicad_sch (KiCad schematic)
At the start: 91 parts, among them J1 12402012E212A, J2 I2S, J3 FRONT, J4 VIDEO1, J5 VIDEO2, J6 VIDEO3, SW1 BOOT, U1 W25Q128JVS, U2 USBLC6-2P6, U3 RP2350A, U4 ADV7391BCPZ, U5 RV-3028-C7, U6 THS7314, Y1 ABM8-272-T3

Commit message: Update with ML2032 battery
Parts:
- removed C21: FG0H104ZF, Library:FG0H104ZF, symbol Device:C_Polarized_Small
- added BT1: ML2032, Library:CR2032-BS-6-1, symbol Device:Battery_Cell
- renumbered C22 to C21, C23 to C22, C24 to C23, C25 to C24, C26 to C25, C27 to C26, C28 to C27, C29 to C28, C30 to C29, C31 to C30, C32 to C31, C33 to C32, C34 to C33, C35 to C34, C36 to C35, C37 to C36
Connections:
- net GND: now also BT1.2 (-)
- net at U5.6 (VBACKUP): now also BT1.1 (+)

Commit message: Small hardware update
Parts:
- added C21: 100n, Capacitor_SMD:C_0603_1608Metric, symbol Device:C_Small
- R10, R9: LCSC C23186 -> C23162
- renumbered C22 to C20, C20 to C22, C21 to C23, C23 to C25, C25 to C26, C26 to C27, C27 to C28, C28 to C29, C29 to C30, C30 to C31, C31 to C32, C32 to C33, C33 to C34, C34 to C35, C35 to C36, C36 to C37
Connections:
- net +1V8: now also C20.1; no longer C30.2, R19.1
- net GND: now also C21.2
- net at BT1.1 (+), U5.6 (VBACKUP): now also C21.1
- net at C22.1, C24.1, FB1.2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: now also C30.2, R19.1; no longer C20.1
Other:
- moved on the sheet: C20, C24

Commit message: Hardware: series inductor for the DAC HF compensation
Add L3 (4.7 uH) and L4 (1.5 uH), both 0805, in series with R15: 6.2 uH
in total, chosen from measurements (4.7+2.2 was too high, 4.7+1.0 too
low). The two existing 1008 coils move to L5/L6. Gerbers, BOM,
positions, netlist and schematic PDF regenerated.
Parts:
- added L3: 4.7uH, Inductor_SMD:L_0805_2012Metric, symbol Device:L_Small
- added L4: 1.5uH, Inductor_SMD:L_0805_2012Metric, symbol Device:L_Small
Connections:
- net GND: now also L4.2; no longer R15.2
- new net: L3.1, R15.2
- new net: L3.2, L4.1
Other:
- moved on the sheet: R15
Changed lines of the file:
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@@
 	)
 	(junction
+		(at 212.09 116.84)
+		(diameter 0)
+		(color 0 0 0 0)
+	)
+	(junction
 		(at 152.4 106.68)
 		(diameter 0)
@@
 	)
 	(junction
-		(at 212.09 116.84)
-		(diameter 0)
-		(color 0 0 0 0)
-	)
-	(junction
 		(at 124.46 26.67)
 		(diameter 0)
@@
 	(wire
 		(pts
+			(xy 212.09 97.79) (xy 212.09 99.06)
+		)
+		(stroke
+			(width 0)
+			(type default)
+		)
+	)
+	(wire
+		(pts
 			(xy 57.15 166.37) (xy 57.15 168.91)
 		)
@@
 	(wire
 		(pts
-			(xy 212.09 91.44) (xy 212.09 101.6)
+			(xy 212.09 91.44) (xy 212.09 92.71)
 		)
 		(stroke
@@
 	(wire
 		(pts
-			(xy 212.09 106.68) (xy 212.09 116.84)
+			(xy 137.16 116.84) (xy 137.16 129.54)
 		)
 		(stroke
@@
 	(wire
 		(pts
-			(xy 137.16 116.84) (xy 137.16 129.54)
+			(xy 104.14 63.5) (xy 109.22 63.5)
 		)
 		(stroke
@@
 	(wire
 		(pts
-			(xy 104.14 63.5) (xy 109.22 63.5)
+			(xy 132.08 58.42) (xy 135.89 58.42)
 		)
 		(stroke
@@
 	(wire
 		(pts
-			(xy 132.08 58.42) (xy 135.89 58.42)
+			(xy 106.68 26.67) (xy 115.57 26.67)
 		)
 		(stroke
@@
 	(wire
 		(pts
-			(xy 106.68 26.67) (xy 115.57 26.67)
+			(xy 184.15 71.12) (xy 184.15 62.23)
 		)
 		(stroke
@@
 	(wire
 		(pts
-			(xy 184.15 71.12) (xy 184.15 62.23)
+			(xy 212.09 104.14) (xy 212.09 105.41)
 		)
 		(stroke
@@
 	(wire
 		(pts
+			(xy 212.09 110.49) (xy 212.09 116.84)
+		)
+		(stroke
+			(width 0)
+			(type default)
+		)
+	)
+	(wire
+		(pts
 			(xy 267.97 135.89) (xy 267.97 140.97)
 		)
@@
 	)
 	(symbol
+		(lib_id "Device:L_Small")
+		(at 212.09 101.6 0)
+		(unit 1)
+		(body_style 1)
+		(exclude_from_sim no)
+		(in_bom yes)
+		(on_board yes)
+		(in_pos_files yes)
+		(dnp no)
+		(property "Reference" "L3"
+			(at 212.852 100.33 0)
+			(show_name no)
+			(do_not_autoplace no)
+			(effects
+				(font
+					(size 1.27 1.27)
+				)
+				(justify left)
+			)
+		)
+		(property "Value" "4.7uH"
+			(at 212.852 102.87 0)
+			(show_name no)
+			(do_not_autoplace no)
+			(effects
+				(font
+					(size 1.27 1.27)
+				)
+				(justify left)
+			)
+		)
+		(property "Footprint" "Inductor_SMD:L_0805_2012Metric"
+			(at 212.09 101.6 0)
+			(hide yes)
+			(show_name no)
+			(do_not_autoplace no)
+			(effects
+				(font
+					(size 1.27 1.27)
+				)
+			)
+		)
+		(property "Datasheet" "0805CS-472"
+			(at 212.09 101.6 0)
+			(hide yes)
+			(show_name no)
+			(do_not_autoplace no)
+			(effects
+				(font
+					(size 1.27 1.27)
+				)
+			)
+		)
+		(property "Description" "Inductor, small symbol"
+			(at 212.09 101.6 0)
+			(hide yes)
+			(show_name no)
+			(do_not_autoplace no)
+			(effects
+				(font
+					(size 1.27 1.27)
+				)
+			)
+		)
+		(property "LCSC" "C9900302166 "
+			(at 212.09 101.6 0)
+			(hide yes)
+			(show_name no)
+			(do_not_autoplace no)
+			(effects
+				(font
+					(size 1.27 1.27)
+				)
+			)
+		)
+		(pin "1"
+		)
+		(pin "2"
+		)
+		(instances
+			(project "PAL-sign"
+				(path "/d14260ee-e09c-47d0-8616-c1f67019dae8"
+					(reference "L3")
+					(unit 1)
+				)
+			)
+		)
+	)
+	(symbol
 		(lib_id "Device:C_Small")
 		(at 264.16 140.97 90)
@@
 	(symbol
 		(lib_id "Device:R_Small")
-		(at 212.09 104.14 0)
+		(at 212.09 95.25 0)
 		(unit 1)
 		(body_style 1)
@@
 		(dnp no)
 		(property "Reference" "R15"
-			(at 214.122 102.87 0)
+			(at 214.122 93.98 0)
 			(show_name no)
 			(do_not_autoplace no)
@@
 		)
 		(property "Value" "300"
-			(at 214.122 104.9021 0)
+			(at 214.122 96.0121 0)
 			(show_name no)
 			(do_not_autoplace no)
@@
 		)
 		(property "Footprint" "Resistor_SMD:R_0603_1608Metric"
-			(at 212.09 104.14 0)
+			(at 212.09 95.25 0)
 			(hide yes)
 			(show_name no)
@@
 		)
 		(property "Datasheet" ""
-			(at 212.09 104.14 0)
+			(at 212.09 95.25 0)
 			(hide yes)
 			(show_name no)
@@
 		)
 		(property "Description" "Resistor, small symbol"
-			(at 212.09 104.14 0)
+			(at 212.09 95.25 0)
 			(hide yes)
 			(show_name no)
@@
 		)
 		(property "LCSC" "C23025"
-			(at 212.09 104.14 0)
+			(at 212.09 95.25 0)
 			(hide yes)
 			(show_name no)
@@
 		)
 		(property "KLC_S3.3" ""
-			(at 212.09 104.14 0)
+			(at 212.09 95.25 0)
 			(hide yes)
 			(show_name no)
@@
 		)
 		(property "KLC_S4.1" ""
-			(at 212.09 104.14 0)
+			(at 212.09 95.25 0)
 			(hide yes)
 			(show_name no)
@@
 		)
 		(property "KLC_S4.2_DVDD" ""
-			(at 212.09 104.14 0)
+			(at 212.09 95.25 0)
 			(hide yes)
 			(show_name no)
@@
 		)
 		(property "KLC_S4.2_VREG_LX" ""
-			(at 212.09 104.14 0)
+			(at 212.09 95.25 0)
 			(hide yes)
 			(show_name no)
@@
 					(unit 1)
 				)
+			)
+		)
+	)
+	(symbol
+		(lib_id "Device:L_Small")
+		(at 212.09 107.95 0)
+		(unit 1)
+		(body_style 1)
+		(exclude_from_sim no)
+		(in_bom yes)
+		(on_board yes)
+		(in_pos_files yes)
+		(dnp no)
+		(property "Reference" "L4"
+			(at 212.852 106.68 0)
+			(show_name no)
+			(do_not_autoplace no)
+			(effects
+				(font
+					(size 1.27 1.27)
+				)
+				(justify left)
+			)
+		)
+		(property "Value" "1.5uH"
+			(at 212.852 109.22 0)
+			(show_name no)
+			(do_not_autoplace no)
+			(effects
+				(font
+					(size 1.27 1.27)
+				)
+				(justify left)
+			)
+		)
+		(property "Footprint" "Inductor_SMD:L_0805_2012Metric"
+			(at 212.09 107.95 0)
+			(hide yes)
+			(show_name no)
+			(do_not_autoplace no)
+			(effects
+				(font
+					(size 1.27 1.27)
+				)
+			)
+		)
+		(property "Datasheet" "0805CS-152"
+			(at 212.09 107.95 0)
+			(hide yes)
+			(show_name no)
+			(do_not_autoplace no)
+			(effects
+				(font
+					(size 1.27 1.27)
+				)
+			)
+		)
+		(property "Description" "Inductor, small symbol"
+			(at 212.09 107.95 0)
+			(hide yes)
+			(show_name no)
+			(do_not_autoplace no)
+			(effects
+				(font
+					(size 1.27 1.27)
+				)
+			)
+		)
+		(property "LCSC" "C41336172 "
+			(at 212.09 107.95 0)
+			(hide yes)
+			(show_name no)
+			(do_not_autoplace no)
+			(effects
+				(font
+					(size 1.27 1.27)
+				)
+			)
+		)
+		(pin "1"
+		)
+		(pin "2"
+		)
+		(instances
+			(project "PAL-sign"
+				(path "/d14260ee-e09c-47d0-8616-c1f67019dae8"
+					(reference "L4")
+					(unit 1)
+				)
