File: Hardware/Kicad/psu.kicad_sch (KiCad schematic)
At the start: 21 parts, among them J7 Barrel_Jack_Switch, U7 TPS62160DSG, U8 TPS7A2033PDBVR, U9 TPS7A2018PDBVR

Commit message: Update PSU, so USB powering works too
Parts:
- removed R25: 10k, Resistor_SMD:R_0603_1608Metric, symbol Device:R_Small
Connections:
- net +5V: now also U8.3 (EN)
- net GND: now also U7.8 (PG)
Changed lines of the file:
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@@
+	)
+	(junction
+		(at 165.1 45.72)
+		(diameter 0)
+		(color 0 0 0 0)
 	)
 	(junction
@@
 	)
 	(junction
+		(at 71.12 55.88)
+		(diameter 0)
+		(color 0 0 0 0)
+	)
+	(junction
 		(at 60.96 45.72)
 		(diameter 0)
@@
 	)
 	(junction
-		(at 137.16 73.66)
-		(diameter 0)
-		(color 0 0 0 0)
-	)
-	(junction
 		(at 194.31 45.72)
 		(diameter 0)
@@
 	(wire
 		(pts
-			(xy 80.01 73.66) (xy 137.16 73.66)
-		)
-		(stroke
-			(width 0)
-			(type default)
-		)
-	)
-	(wire
-		(pts
 			(xy 156.21 52.07) (xy 156.21 45.72)
 		)
@@
 	(wire
 		(pts
-			(xy 156.21 45.72) (xy 166.37 45.72)
+			(xy 156.21 45.72) (xy 165.1 45.72)
 		)
 		(stroke
@@
 	(wire
 		(pts
-			(xy 137.16 73.66) (xy 165.1 73.66)
-		)
-		(stroke
-			(width 0)
-			(type default)
-		)
-	)
-	(wire
-		(pts
 			(xy 241.3 34.29) (xy 241.3 45.72)
 		)
@@
 	(wire
 		(pts
+			(xy 165.1 45.72) (xy 166.37 45.72)
+		)
+		(stroke
+			(width 0)
+			(type default)
+		)
+	)
+	(wire
+		(pts
 			(xy 102.87 45.72) (xy 106.68 45.72)
 		)
@@
 	(wire
 		(pts
-			(xy 71.12 54.61) (xy 71.12 58.42)
+			(xy 71.12 54.61) (xy 71.12 55.88)
 		)
 		(stroke
@@
 	(wire
 		(pts
-			(xy 80.01 55.88) (xy 82.55 55.88)
-		)
-		(stroke
-			(width 0)
-			(type default)
-		)
-	)
-	(wire
-		(pts
 			(xy 194.31 26.67) (xy 194.31 35.56)
 		)
@@
 	(wire
 		(pts
-			(xy 137.16 57.15) (xy 137.16 73.66)
+			(xy 165.1 45.72) (xy 165.1 48.26)
 		)
 		(stroke
@@
 	(wire
 		(pts
-			(xy 165.1 48.26) (xy 165.1 73.66)
-		)
-		(stroke
-			(width 0)
-			(type default)
-		)
-	)
-	(wire
-		(pts
 			(xy 241.3 57.15) (xy 241.3 58.42)
 		)
@@
 	(wire
 		(pts
+			(xy 71.12 55.88) (xy 82.55 55.88)
+		)
+		(stroke
+			(width 0)
+			(type default)
+		)
+	)
+	(wire
+		(pts
 			(xy 184.15 45.72) (xy 184.15 52.07)
 		)
@@
 	(wire
 		(pts
+			(xy 71.12 55.88) (xy 71.12 58.42)
+		)
+		(stroke
+			(width 0)
+			(type default)
+		)
+	)
+	(wire
+		(pts
 			(xy 71.12 45.72) (xy 71.12 49.53)
 		)
@@
 	(wire
 		(pts
-			(xy 137.16 45.72) (xy 137.16 52.07)
-		)
-		(stroke
-			(width 0)
-			(type default)
-		)
-	)
-	(wire
-		(pts
 			(xy 43.18 45.72) (xy 50.8 45.72)
-		)
-		(stroke
-			(width 0)
-			(type default)
-		)
-	)
-	(wire
-		(pts
-			(xy 80.01 73.66) (xy 80.01 55.88)
 		)
 		(stroke
@@
 					(unit 1)
 				)
-			)
-		)
-	)
-	(symbol
-		(lib_id "Device:R_Small")
-		(at 137.16 54.61 0)
-		(unit 1)
-		(body_style 1)
-		(exclude_from_sim no)
-		(in_bom yes)
-		(on_board yes)
-		(in_pos_files yes)
-		(dnp no)
-		(fields_autoplaced yes)
-		(property "Reference" "R25"
-			(at 139.7 53.3399 0)
-			(show_name no)
-			(do_not_autoplace no)
-			(effects
-				(font
-					(size 1.27 1.27)
-				)
-				(justify left)
-			)
-		)
-		(property "Value" "10k"
-			(at 139.7 55.8799 0)
-			(show_name no)
-			(do_not_autoplace no)
-			(effects
-				(font
-					(size 1.27 1.27)
-				)
-				(justify left)
-			)
-		)
-		(property "Footprint" "Resistor_SMD:R_0603_1608Metric"
-			(at 137.16 54.61 0)
-			(hide yes)
-			(show_name no)
-			(do_not_autoplace no)
-			(effects
-				(font
-					(size 1.27 1.27)
-				)
-			)
-		)
-		(property "Datasheet" ""
-			(at 137.16 54.61 0)
-			(hide yes)
-			(show_name no)
-			(do_not_autoplace no)
-			(effects
-				(font
-					(size 1.27 1.27)
-				)
-			)
-		)
-		(property "Description" "Resistor, small symbol"
-			(at 137.16 54.61 0)
-			(hide yes)
-			(show_name no)
-			(do_not_autoplace no)
-			(effects
-				(font
-					(size 1.27 1.27)
-				)
-			)
-		)
-		(property "LCSC" "C25804"
-			(at 137.16 54.61 0)
-			(hide yes)
-			(show_name no)
-			(do_not_autoplace no)
-			(effects
-				(font
-					(size 1.27 1.27)
-				)
-			)
-		)
-		(property "KLC_S3.3" ""
-			(at 137.16 54.61 0)
-			(hide yes)
-			(show_name no)
-			(do_not_autoplace no)
-			(effects
-				(font
-					(size 1.27 1.27)
-				)
-			)
-		)
-		(property "KLC_S4.1" ""
-			(at 137.16 54.61 0)
-			(hide yes)
-			(show_name no)
-			(do_not_autoplace no)
-			(effects
-				(font
-					(size 1.27 1.27)
-				)
-			)
-		)
-		(property "KLC_S4.2_DVDD" ""
-			(at 137.16 54.61 0)
-			(hide yes)
-			(show_name no)
-			(do_not_autoplace no)
-			(effects
-				(font
-					(size 1.27 1.27)
-				)
-			)
-		)
-		(property "KLC_S4.2_VREG_LX" ""
-			(at 137.16 54.61 0)
-			(hide yes)
-			(show_name no)
-			(do_not_autoplace no)
-			(effects
-				(font
-					(size 1.27 1.27)
-				)
-			)
-		)
-		(pin "1"
-		)
-		(pin "2"
-		)
-		(instances
-			(project "PAL-sign"
-				(path "/5e4b4b86-505e-4573-b1db-0e4430e7f8ee"
-					(reference "R25")
-					(unit 1)
-				)
-			)
-			(project "psu"
-				(path "/8e3ad6b7-1e34-483c-9952-fb6d399791d2"
-					(reference "R25")
-					(unit 1)
-				)

Commit message: Hardware: series inductor for the DAC HF compensation
Add L3 (4.7 uH) and L4 (1.5 uH), both 0805, in series with R15: 6.2 uH
in total, chosen from measurements (4.7+2.2 was too high, 4.7+1.0 too
low). The two existing 1008 coils move to L5/L6. Gerbers, BOM,
positions, netlist and schematic PDF regenerated.
Parts:
- renumbered L3 to L5, L4 to L6
Changed lines of the file:
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@@
 		(in_pos_files yes)
 		(dnp no)
-		(property "Reference" "L3"
+		(property "Reference" "L5"
 			(at 109.22 40.894 90)
 			(show_name no)
@@
 			(project "PAL-sign"
 				(path "/5e4b4b86-505e-4573-b1db-0e4430e7f8ee"
-					(reference "L3")
+					(reference "L5")
 					(unit 1)
 				)
@@
 		(in_pos_files yes)
 		(dnp no)
-		(property "Reference" "L4"
+		(property "Reference" "L6"
 			(at 130.81 40.894 90)
 			(show_name no)
@@
 			(project "PAL-sign"
 				(path "/5e4b4b86-505e-4573-b1db-0e4430e7f8ee"
-					(reference "L4")
+					(reference "L6")
 					(unit 1)
 				)
